Commit message: 202405122117

File: multisections.urdf (robot description, URDF)
Before this commit: robot snake_robot_cit, 11 links, 10 joints
Links:
- link base_link: geometry collision mesh filename=package://snake_robot_cit_notail_description/meshes/base_li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 scale=0.001 0.001 0.001; visual mesh filename=package://snake_robot_cit_notail_description/meshes/base_li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 scale=0.001 0.001 0.001
- link onemodule1_1: geometry collision mesh filename=package://snake_robot_cit_notail_description/meshes/onemodu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 scale=0.001 0.001 0.001; visual mesh filename=package://snake_robot_cit_notail_description/meshes/onemodu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 scale=0.001 0.001 0.001
- link onemodule2_1: geometry collision mesh filename=package://snake_robot_cit_notail_description/meshes/onemodu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 scale=0.001 0.001 0.001; visual mesh filename=package://snake_robot_cit_notail_description/meshes/onemodu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 scale=0.001 0.001 0.001
- link onemodule3_1: geometry collision mesh filename=package://snake_robot_cit_notail_description/meshes/onemodu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 scale=0.001 0.001 0.001; visual mesh filename=package://snake_robot_cit_notail_description/meshes/onemodu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 scale=0.001 0.001 0.001
- link onemodule4_1: geometry collision mesh filename=package://snake_robot_cit_notail_description/meshes/onemodu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 scale=0.001 0.001 0.001; visual mesh filename=package://snake_robot_cit_notail_description/meshes/onemodu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 scale=0.001 0.001 0.001
- link onemodule5_1: geometry collision mesh filename=package://snake_robot_cit_notail_description/meshes/onemodu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 scale=0.001 0.001 0.001; visual mesh filename=package://snake_robot_cit_notail_description/meshes/onemodu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 scale=0.001 0.001 0.001
- link onemodule6_1: geometry collision mesh filename=package://snake_robot_cit_notail_description/meshes/onemodu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 scale=0.001 0.001 0.001; visual mesh filename=package://snake_robot_cit_notail_description/meshes/onemodu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 scale=0.001 0.001 0.001
- link onemodule7_1: geometry collision mesh filename=package://snake_robot_cit_notail_description/meshes/onemodu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 scale=0.001 0.001 0.001; visual mesh filename=package://snake_robot_cit_notail_description/meshes/onemodu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 scale=0.001 0.001 0.001
- link onemodule8_1: geometry collision mesh filename=package://snake_robot_cit_notail_description/meshes/onemodu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 scale=0.001 0.001 0.001; visual mesh filename=package://snake_robot_cit_notail_description/meshes/onemodu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 scale=0.001 0.001 0.001
- link onemodule9_1: geometry collision mesh filename=package://snake_robot_cit_notail_description/meshes/onemodu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 scale=0.001 0.001 0.001; visual mesh filename=package://snake_robot_cit_notail_description/meshes/onemodu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 scale=0.001 0.001 0.001
- link tailmodule_1: mass 2.1589988659404105 -> 2.1365597828004343; geometry collision mesh filename=package://snake_robot_cit_notail_description/meshes/tailmod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 scale=0.001 0.001 0.001; visual mesh filename=package://snake_robot_cit_notail_description/meshes/tailmod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 scale=0.001 0.001 0.001
